File: motor monitor pcb /motor monitor pcb.kicad_sch (KiCad schematic)
At the start: 11 parts, among them J1 Motor_Out, J2 Power_In, U1 ESP32-WROOM-32, U2 MPU-6050, U3 L298N

Commit message: Add PCB layout - components placed
Footprints assigned, board outline set, all components
placed and ready for routing. Schematic also finalized
with RC anti-aliasing filter added.
Parts:
- C1, C2, C3, C4, C5: footprint (none) -> Capacitor_THT:C_Disc_D5.0mm_W2.5mm_P5.00mm
- J1, J2: footprint (none) -> Connector_PinHeader_2.54mm:PinHeader_1x02_P2.54mm_Vertical
- R1: footprint (none) -> Resistor_THT:R_Axial_DIN0207_L6.3mm_D2.5mm_P10.16mm_Horizontal
Other:
- moved on the sheet: C1
Changed lines of the file:
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@@
 	(wire
 		(pts
-			(xy 242.57 57.15) (xy 241.3 57.15)
+			(xy 234.95 57.15) (xy 233.68 57.15)
 		)
 		(stroke
@@
 	(wire
 		(pts
-			(xy 242.57 48.26) (xy 242.57 57.15)
+			(xy 234.95 48.26) (xy 234.95 57.15)
 		)
 		(stroke
@@
 	(wire
 		(pts
-			(xy 242.57 33.02) (xy 242.57 40.64)
+			(xy 234.95 33.02) (xy 234.95 40.64)
 		)
 		(stroke
@@
 			)
 		)
-		(property "Footprint" ""
+		(property "Footprint" "Capacitor_THT:C_Disc_D5.0mm_W2.5mm_P5.00mm"
 			(at 75.8952 45.72 0)
 			(hide yes)
@@
 			)
 		)
-		(property "Footprint" ""
+		(property "Footprint" "Capacitor_THT:C_Disc_D5.0mm_W2.5mm_P5.00mm"
 			(at 131.7752 52.07 0)
 			(hide yes)
@@
 			)
 		)
-		(property "Footprint" ""
+		(property "Footprint" "Capacitor_THT:C_Disc_D5.0mm_W2.5mm_P5.00mm"
 			(at 213.0552 125.73 0)
 			(hide yes)
@@
 			)
 		)
-		(property "Footprint" ""
+		(property "Footprint" "Resistor_THT:R_Axial_DIN0207_L6.3mm_D2.5mm_P10.16mm_Horizontal"
 			(at 200.66 116.332 90)
 			(hide yes)
@@
 			)
 		)
-		(property "Footprint" ""
+		(property "Footprint" "Capacitor_THT:C_Disc_D5.0mm_W2.5mm_P5.00mm"
 			(at 204.1652 41.91 0)
 			(hide yes)
@@
 	(symbol
 		(lib_id "power:VCC")
-		(at 242.57 33.02 0)
+		(at 234.95 33.02 0)
 		(unit 1)
 		(body_style 1)
@@
 		(fields_autoplaced yes)
 		(property "Reference" "#PWR08"
-			(at 242.57 36.83 0)
+			(at 234.95 36.83 0)
 			(hide yes)
 			(show_name no)
@@
 		)
 		(property "Value" "VCC"
-			(at 242.57 27.94 0)
+			(at 234.95 27.94 0)
 			(show_name no)
 			(do_not_autoplace no)
@@
 		)
 		(property "Footprint" ""
-			(at 242.57 33.02 0)
+			(at 234.95 33.02 0)
 			(hide yes)
 			(show_name no)
@@
 		)
 		(property "Datasheet" ""
-			(at 242.57 33.02 0)
+			(at 234.95 33.02 0)
 			(hide yes)
 			(show_name no)
@@
 		)
 		(property "Description" "Power symbol creates a global label with name \"VCC\""
-			(at 242.57 33.02 0)
+			(at 234.95 33.02 0)
 			(hide yes)
 			(show_name no)
@@
 	(symbol
 		(lib_id "power:GND")
-		(at 241.3 57.15 0)
+		(at 233.68 57.15 0)
 		(unit 1)
 		(body_style 1)
@@
 		(fields_autoplaced yes)
 		(property "Reference" "#PWR06"
-			(at 241.3 63.5 0)
+			(at 233.68 63.5 0)
 			(hide yes)
 			(show_name no)
@@
 		)
 		(property "Value" "GND"
-			(at 241.3 62.23 0)
+			(at 233.68 62.23 0)
 			(show_name no)
 			(do_not_autoplace no)
@@
 		)
 		(property "Footprint" ""
-			(at 241.3 57.15 0)
+			(at 233.68 57.15 0)
 			(hide yes)
 			(show_name no)
@@
 		)
 		(property "Datasheet" ""
-			(at 241.3 57.15 0)
+			(at 233.68 57.15 0)
 			(hide yes)
 			(show_name no)
@@
 		)
 		(property "Description" "Power symbol creates a global label with name \"GND\" , ground"
-			(at 241.3 57.15 0)
+			(at 233.68 57.15 0)
 			(hide yes)
 			(show_name no)
@@
 			)
 		)
-		(property "Footprint" ""
+		(property "Footprint" "Connector_PinHeader_2.54mm:PinHeader_1x02_P2.54mm_Vertical"
 			(at 252.73 83.82 0)
 			(hide yes)
@@
 			)
 		)
-		(property "Footprint" ""
+		(property "Footprint" "Connector_PinHeader_2.54mm:PinHeader_1x02_P2.54mm_Vertical"
 			(at 257.81 101.6 0)
 			(hide yes)
@@
 	(symbol
 		(lib_id "Device:C")
-		(at 242.57 44.45 0)
+		(at 234.95 44.45 0)
 		(unit 1)
 		(body_style 1)
@@
 		(fields_autoplaced yes)
 		(property "Reference" "C1"
-			(at 246.38 43.1799 0)
+			(at 238.76 43.1799 0)
 			(show_name no)
 			(do_not_autoplace no)
@@
 		)
 		(property "Value" "100nF"
-			(at 246.38 45.7199 0)
+			(at 238.76 45.7199 0)
 			(show_name no)
 			(do_not_autoplace no)
@@
 			)
 		)
-		(property "Footprint" ""
-			(at 243.5352 48.26 0)
+		(property "Footprint" "Capacitor_THT:C_Disc_D5.0mm_W2.5mm_P5.00mm"
+			(at 235.9152 48.26 0)
 			(hide yes)
 			(show_name no)
@@
 		)
 		(property "Datasheet" ""
-			(at 242.57 44.45 0)
+			(at 234.95 44.45 0)
 			(hide yes)
 			(show_name no)
@@
 		)
 		(property "Description" "Unpolarized capacitor"
-			(at 242.57 44.45 0)
-			(hide yes)
-			(show_name no)
+			(at 234.95 44.45 0)
+			(hide yes)
+			(show_name no)
