File: motor monitor pcb /motor monitor pcb.kicad_pcb (KiCad board)
At the start: 2 copper layers, 100 x 80 mm, 11 parts, among them J1 Motor_Out, J2 Power_In, U1 ESP32-WROOM-32, U2 MPU-6050, U3 L298N

Commit message: PCB routing in progress
Routing:
- net GND: track 0.00 -> 181.9 mm
- net VCC: track 0.00 -> 121.5 mm
- net /SCL: track 0.00 -> 85.1 mm
- net Net-(U1-IO14): track 0.00 -> 82.9 mm
- net Net-(U1-IO26): track 0.00 -> 65.4 mm, vias 0 -> 1
- net /ADC_MOTOR: track 0.00 -> 63.1 mm, vias 0 -> 2
- net /SDA: track 0.00 -> 61.9 mm, vias 0 -> 2
- net Net-(U1-IO27): track 0.00 -> 61.5 mm
- net /SENSE_A: track 0.00 -> 41.3 mm
- net /MOTOR_A: track 0.00 -> 35.9 mm, vias 0 -> 1
- net /MOTOR_B: track 0.00 -> 29.0 mm, vias 0 -> 2

Commit message: fixes in pcb layout
Routing:
- net /SCL: track 85.1 -> 58.6 mm
- net VCC: track 121.5 -> 125.2 mm
- net /ADC_MOTOR: track 63.1 -> 64.8 mm, vias 2 -> 1
- net /SDA: track 61.9 -> 61.4 mm, vias 2 -> 0
Changed lines of the file:
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@@
-	)
-	(segment
-		(start 58.035 69.965)
-		(end 63.45 69.965)
-		(width 0.5)
-		(layer "F.Cu")
-		(net "VCC")
 	)
 	(segment
@@
 	)
 	(segment
-		(start 63.45 69.965)
-		(end 63.45 71.765)
+		(start 65.835 69.965)
+		(end 63.665 72.135)
+		(width 0.5)
+		(layer "F.Cu")
+		(net "VCC")
+	)
+	(segment
+		(start 76.415 72.1)
+		(end 78.95 69.565)
 		(width 0.5)
 		(layer "F.Cu")
@@
 	)
 	(segment
-		(start 76.38 72.135)
-		(end 78.95 69.565)
+		(start 78.95 69.565)
+		(end 98.304542 69.565)
 		(width 0.5)
 		(layer "F.Cu")
@@
 	)
 	(segment
+		(start 24.5 58.46)
+		(end 38.94 72.9)
+		(width 0.5)
+		(layer "F.Cu")
+		(net "VCC")
+	)
+	(segment
+		(start 30.08 112.85)
+		(end 28.81 112.85)
+		(width 0.5)
+		(layer "F.Cu")
+		(net "VCC")
+	)
+	(segment
+		(start 62.285 72.1)
+		(end 76.415 72.1)
+		(width 0.5)
+		(layer "F.Cu")
+		(net "VCC")
+	)
+	(segment
+		(start 27.46 106.46)
+		(end 25.5 104.5)
+		(width 0.5)
+		(layer "F.Cu")
+		(net "VCC")
+	)
+	(segment
+		(start 63.665 72.135)
+		(end 62.25 72.135)
+		(width 0.5)
+		(layer "F.Cu")
+		(net "VCC")
+	)
+	(segment
+		(start 58.035 69.965)
+		(end 65.835 69.965)
+		(width 0.5)
+		(layer "F.Cu")
+		(net "VCC")
+	)
+	(segment
+		(start 112 59)
+		(end 111.65 59.35)
+		(width 0.5)
+		(layer "F.Cu")
+		(net "VCC")
+	)
+	(segment
+		(start 62.25 72.135)
+		(end 62.285 72.1)
+		(width 0.5)
+		(layer "F.Cu")
+		(net "VCC")
+	)
+	(segment
+		(start 38.94 72.9)
+		(end 54.9 72.9)
+		(width 0.5)
+		(layer "F.Cu")
+		(net "VCC")
+	)
+	(segment
 		(start 55 73)
 		(end 58.035 69.965)
@@
 	)
 	(segment
-		(start 30.08 112.85)
-		(end 28.81 112.85)
-		(width 0.5)
-		(layer "F.Cu")
-		(net "VCC")
-	)
-	(segment
-		(start 24.5 58.46)
-		(end 39.04 73)
-		(width 0.5)
-		(layer "F.Cu")
-		(net "VCC")
-	)
-	(segment
-		(start 78.95 69.565)
-		(end 98.304542 69.565)
-		(width 0.5)
-		(layer "F.Cu")
-		(net "VCC")
-	)
-	(segment
-		(start 27.46 106.46)
-		(end 25.5 104.5)
-		(width 0.5)
-		(layer "F.Cu")
-		(net "VCC")
-	)
-	(segment
-		(start 39.04 73)
+		(start 54.9 72.9)
 		(end 55 73)
-		(width 0.5)
-		(layer "F.Cu")
-		(net "VCC")
-	)
-	(segment
-		(start 63.08 72.135)
-		(end 62.25 72.135)
-		(width 0.5)
-		(layer "F.Cu")
-		(net "VCC")
-	)
-	(segment
-		(start 62.25 72.135)
-		(end 76.38 72.135)
-		(width 0.5)
-		(layer "F.Cu")
-		(net "VCC")
-	)
-	(segment
-		(start 112 59)
-		(end 111.65 59.35)
-		(width 0.5)
-		(layer "F.Cu")
-		(net "VCC")
-	)
-	(segment
-		(start 63.45 71.765)
-		(end 63.08 72.135)
 		(width 0.5)
 		(layer "F.Cu")
@@
 	)
 	(segment
-		(start 78.675 73.9)
-		(end 78.675 88.15)
-		(width 0.25)
-		(layer "F.Cu")
-		(net "/SCL")
-	)
-	(segment
 		(start 79.75 73.405)
 		(end 79.905 73.405)
@@
 	)
 	(segment
-		(start 79.275 73.3)
-		(end 78.675 73.9)
-		(width 0.25)
-		(layer "F.Cu")
-		(net "/SCL")
-	)
-	(segment
 		(start 107.25 55.557236)
 		(end 107.25 56.05)
@@
 	)
 	(segment
-		(start 78.675 88.15)
-		(end 90.077387 88.15)
-		(width 0.25)
-		(layer "F.Cu")
-		(net "/SCL")
-	)
-	(segment
 		(start 114.890991 55.3)
 		(end 107.507236 55.3)
@@
 	)
 	(segment
+		(start 79.75 77.215)
+		(end 101.012387 77.215)
+		(width 0.25)
+		(layer "F.Cu")
+		(net "/SDA")
+	)
+	(segment
+		(start 118.575 58.347613)
+		(end 115.077387 54.85)
+		(width 0.25)
+		(layer "F.Cu")
+		(net "/SDA")
+	)
+	(segment
+		(start 107.052556 54.85)
+		(end 106.75 55.152556)
+		(width 0.25)
+		(layer "F.Cu")
+		(net "/SDA")
+	)
+	(segment
+		(start 106.75 55.152556)
+		(end 106.75 55.757191)
+		(width 0.25)
+		(layer "F.Cu")
+		(net "/SDA")
+	)
+	(segment
 		(start 118.575 59.652387)
 		(end 118.575 58.347613)
@@
 	)
 	(segment
+		(start 101.012387 77.215)
+		(end 118.575 59.652387)
+		(width 0.25)
+		(layer "F.Cu")
+		(net "/SDA")
+	)
+	(segment
 		(start 115.077387 54.85)
 		(end 107.052556 54.85)
 		(width 0.25)
 		(layer "F.Cu")
-		(net "/SDA")
-	)
-	(segment
-		(start 101.012387 77.215)
-		(end 118.575 59.652387)
-		(width 0.25)
-		(layer "F.Cu")
-		(net "/SDA")
-	)
-	(segment
-		(start 79.75 77.215)
-		(end 101.012387 77.215)
-		(width 0.25)
-		(layer "F.Cu")
-		(net "/SDA")
-	)
-	(segment
-		(start 118.575 58.347613)
-		(end 115.077387 54.85)
-		(width 0.25)
-		(layer "F.Cu")
-		(net "/SDA")
-	)
-	(segment
-		(start 106.5 55.402556)
-		(end 106.5 56.007191)
-		(width 0.25)
-		(layer "F.Cu")
-		(net "/SDA")
-	)
-	(segment
-		(start 107.052556 54.85)
-		(end 106.5 55.402556)
-		(width 0.25)
-		(layer "F.Cu")
-		(net "/SDA")
-	)
-	(via
-		(at 106.5 56.007191)
-		(size 0.8)
-		(drill 0.4)
-		(layers "F.Cu" "B.Cu")
-		(net "/SDA")
-	)
-	(via
-		(at 79.75 77.215)
-		(size 0.6)
-		(drill 0.3)
-		(layers "F.Cu" "B.Cu")
-		(net "/SDA")
-	)
-	(segment
-		(start 79.75 77.25)
-		(end 79.8 77.3)
-		(width 0.25)
-		(layer "B.Cu")
-		(net "/SDA")
-	)
-	(segment
-		(start 79.75 77.215)
-		(end 79.75 77.25)
-		(width 0.25)
-		(layer "B.Cu")
 		(net "/SDA")
 	)
@@
 		(net "/ADC_MOTOR")
 	)
-	(via
-		(at 58.5 95.5)
-		(size 0.6)
-		(drill 0.3)
-		(layers "F.Cu" "B.Cu")
-		(net "/ADC_MOTOR")
-	)
-	(segment
-		(start 66.789442 101.289442)
-		(end 61 95.5)
+	(segment
+		(start 58.5 95.2)
+		(end 60.7 95.2)
 		(width 0.25)
 		(layer "B.Cu")
@@
 	)
 	(segment
-		(start 61 95.5)
-		(end 58.5 95.5)
+		(start 58.5 96)
+		(end 58.5 95.2)
 		(width 0.25)
 		(layer "B.Cu")
+		(net "/ADC_MOTOR")
+	)
+	(segment
+		(start 58 96.5)
+		(end 58.5 96)
+		(width 0.25)
+		(layer "B.Cu")
+		(net "/ADC_MOTOR")
+	)
+	(segment
+		(start 60.7 95.2)
+		(end 66.789442 101.289442)
+		(width 0.25)
+		(layer "B.Cu")
